File: lumacode2rgb/LumaCode2RGBBoard/input.kicad_sch (KiCad schematic)
At the start: 38 parts, among them J1 Conn_01x07, J2 Conn_01x12, J3 AudioJack3, U1 TVP7002, U2 AP2127K-3.3, U3 AP2127K-3.3, U4 AP2127K-1.9, U5 AP2127K-1.9, U6 AP2127K-1.9

Commit message: Schematic and start PCB layout
Parts:
- removed J1: Conn_01x07, Connector_PinHeader_2.54mm:PinHeader_1x07_P2.54mm_Vertical, symbol Connector_Generic:Conn_01x07
- removed J2: Conn_01x12, Connector_PinHeader_2.54mm:PinHeader_1x12_P2.54mm_Vertical, symbol Connector_Generic:Conn_01x12
- removed JAUDIO1: Conn_Coaxial, symbol Connector:Conn_Coaxial
- removed JP1: SolderJumper_2_Open, Jumper:SolderJumper-2_P1.3mm_Open_RoundedPad1.0x1.5mm, symbol Jumper:SolderJumper_2_Open
- added JBOTTOM1, JBOTTOM2: Conn_01x10, Connector_PinHeader_2.54mm:PinHeader_1x10_P2.54mm_Vertical, symbol Connector_Generic:Conn_01x10
- added R5: 10k, Resistor_SMD:R_0805_2012Metric, symbol Device:R_Small
- added SW1: SW_Push, Button_Switch_THT:SW_Tactile_SKHH_Angled, symbol Switch:SW_Push
- JAUDIO1: renamed from J3; footprint Connector_Audio:Jack_3.5mm_CUI_SJ-3523-SMT_Horizontal -> Connector_Audio:Jack_3.5mm_Lumberg_1503_07_Horizontal
- JLUMACODE1: footprint (none) -> footprints:RCA_JACK
- U1: footprint Package_QFP:TQFP-100_14x14mm_P0.5mm -> Package_QFP:TQFP-100-1EP_14x14mm_P0.5mm_EP5x5mm
Connections:
- net +5V: now also JBOTTOM2.5 (Pin_5)
- net AUDIO_GND: now also JBOTTOM2.1 (Pin_1)
- net AUDIO_LEFT: now also JBOTTOM2.3 (Pin_3)
- net AUDIO_RIGHT: now also JBOTTOM2.2 (Pin_2)
- net CLK: now also JBOTTOM1.10 (Pin_10)
- net G0: now also JBOTTOM1.1 (Pin_1)
- net G1: now also JBOTTOM1.2 (Pin_2)
- net G2: now also JBOTTOM1.3 (Pin_3)
- net G3: now also JBOTTOM1.4 (Pin_4)
- net G4: now also JBOTTOM1.5 (Pin_5)
- net G5: now also JBOTTOM1.6 (Pin_6)
- net G6: now also JBOTTOM1.7 (Pin_7)
- net G7: now also JBOTTOM1.8 (Pin_8)
- net GND: now also JBOTTOM1.9 (Pin_9), JBOTTOM2.4 (Pin_4), SW1.2
- net HSOUT: now also JBOTTOM2.9 (Pin_9)
- net IOVDD: now also R5.2
- net SCL: now also JBOTTOM2.7 (Pin_7)
- net SDA: now also JBOTTOM2.6 (Pin_6)
- net VSOUT: now also JBOTTOM2.8 (Pin_8)
- new net: JBOTTOM2.10 (Pin_10), R5.1, SW1.1
Other:
- moved on the sheet: JAUDIO1

Commit message: PCB layout
Parts:
- removed C20: 10uF, Capacitor_SMD:C_0805_2012Metric, symbol Device:C_Small
Changed lines of the file:
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@@
-    (pin "2")
-  )
-  (symbol (lib_id "Device:C_Small") (at 262.89 76.2 0) (unit 1)
-    (in_bom yes) (on_board yes) (fields_autoplaced)
-    (property "Reference" "C20" (id 0) (at 265.43 74.9362 0)
-      (effects (font (size 1.27 1.27)) (justify left))
-    )
-    (property "Value" "10uF" (id 1) (at 265.43 77.4762 0)
-      (effects (font (size 1.27 1.27)) (justify left))
-    )
-    (property "Footprint" "Capacitor_SMD:C_0805_2012Metric" (id 2) (at 262.89 76.2 0)
-      (effects (font (size 1.27 1.27)) hide)
-    )
-    (property "Datasheet" "~" (id 3) (at 262.89 76.2 0)
-      (effects (font (size 1.27 1.27)) hide)
-    )
-    (pin "1")
     (pin "2")
   )

Commit message: Squeeze all components onto the PCB
Connections:
- net +5V renamed 5V
Changed lines of the file:
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@@
     (stroke (width 0) (type default) (color 0 0 0 0))
   )
-  (wire (pts (xy 241.3 21.59) (xy 241.3 26.67))
+  (wire (pts (xy 241.3 20.32) (xy 241.3 26.67))
     (stroke (width 0) (type default) (color 0 0 0 0))
   )
@@
     (stroke (width 0) (type default) (color 0 0 0 0))
   )
-  (wire (pts (xy 172.72 20.32) (xy 172.72 21.59))
+  (wire (pts (xy 172.72 20.32) (xy 172.72 26.67))
     (stroke (width 0) (type default) (color 0 0 0 0))
   )
@@
     (stroke (width 0) (type default) (color 0 0 0 0))
   )
+  (label "5V" (at 172.72 26.67 90)
+    (effects (font (size 1.27 1.27)) (justify left bottom))
+  )
   (label "AUDIO_LEFT" (at 148.59 25.4 0)
     (effects (font (size 1.27 1.27)) (justify left bottom))
@@
   (label "VSOUT" (at 69.85 125.73 0)
     (effects (font (size 1.27 1.27)) (justify left bottom))
+  )
+  (label "5V" (at 241.3 20.32 270)
+    (effects (font (size 1.27 1.27)) (justify right bottom))
   )
   (label "G4" (at 143.51 162.56 270)
@@
     )
     (property "Datasheet" "" (id 3) (at 241.3 129.54 0)
-      (effects (font (size 1.27 1.27)) hide)
-    )
-    (pin "1")
-  )
-  (symbol (lib_id "power:+5V") (at 241.3 21.59 0) (unit 1)
-    (in_bom yes) (on_board yes) (fields_autoplaced)
-    (property "Reference" "#PWR046" (id 0) (at 241.3 25.4 0)
-      (effects (font (size 1.27 1.27)) hide)
-    )
-    (property "Value" "+5V" (id 1) (at 241.3 16.51 0))
-    (property "Footprint" "" (id 2) (at 241.3 21.59 0)
-      (effects (font (size 1.27 1.27)) hide)
-    )
-    (property "Datasheet" "" (id 3) (at 241.3 21.59 0)
       (effects (font (size 1.27 1.27)) hide)
     )
@@
       (effects (font (size 1.27 1.27)) hide)
     )
-    (pin "1")
-  )
-  (symbol (lib_id "power:+5V") (at 172.72 21.59 180) (unit 1)
-    (in_bom yes) (on_board yes)
-    (property "Reference" "#PWR045" (id 0) (at 172.72 17.78 0)
-      (effects (font (size 1.27 1.27)) hide)
-    )
-    (property "Value" "+5V" (id 1) (at 172.72 26.67 90))
-    (property "Footprint" "" (id 2) (at 172.72 21.59 0)
-      (effects (font (size 1.27 1.27)) hide)
-    )
-    (property "Datasheet" "" (id 3) (at 172.72 21.59 0)
-      (effects (font (size 1.27 1.27)) hide)
-    )
