File: lumacode2rgb/LumaCode2RGBBoard/processing.kicad_sch (KiCad schematic)
At the start: 38 parts, among them J4 USB_B_Micro, J5 Conn_01x07, J6 Conn_01x12, SW1 SW_Push, U10 AP2127K-3.3, U11 74AHC595, U12 74AHC595, U7 PIC16F1455-IML, U8 MachXO2-1200, U9 AP2127K-3.3

Commit message: Schematic and start PCB layout
Parts:
- removed J5: Conn_01x07, Connector_PinHeader_2.54mm:PinHeader_1x07_P2.54mm_Vertical, symbol Connector_Generic:Conn_01x07
- removed J6: Conn_01x12, Connector_PinHeader_2.54mm:PinHeader_1x12_P2.54mm_Vertical, symbol Connector_Generic:Conn_01x12
- removed JPICKIT1: Conn_01x06, Connector_PinHeader_2.54mm:PinHeader_1x06_P2.54mm_Vertical, symbol Connector_Generic:Conn_01x06
- removed R5: 10k, Resistor_SMD:R_0805_2012Metric, symbol Device:R_Small
- removed SW1: SW_Push, Button_Switch_THT:SW_Tactile_SKHH_Angled, symbol Switch:SW_Push
- added JPICKIT1: Conn_01x05, Connector_PinHeader_2.54mm:PinHeader_1x05_P2.54mm_Vertical, symbol Connector_Generic:Conn_01x05
- added JTOP1, JTOP2: Conn_01x10, Connector_PinHeader_2.54mm:PinHeader_1x10_P2.54mm_Vertical, symbol Connector_Generic:Conn_01x10
- J4: footprint Connector_USB:USB_Micro-B_Molex-105017-0001 -> footprints:USB_Micro-B_Amphenol_10104110_Horizontal
- JRGB1: footprint (none) -> footprints:SCART_Edge_mount
- U7: footprint Package_DFN_QFN:HVQFN-16-1EP_3x3mm_P0.5mm_EP1.5x1.5mm -> Package_DFN_QFN:QFN-16-1EP_4x4mm_P0.65mm_EP2.1x2.1mm
- U8: footprint Package_DFN_QFN:QFN-32-1EP_5x5mm_P0.5mm_EP3.6x3.6mm_ThermalVias -> footprints:QFN-32-1EP_5x5mm_P0.5mm_EP3.1x3.1mm_ThermalVias
Connections:
- net +3.3V: now also JPICKIT1.2 (Pin_2)
- net +5V: now also JTOP2.5 (Pin_5)
- net AUDIO_GND: now also JTOP2.1 (Pin_1)
- net AUDIO_LEFT: now also JTOP2.3 (Pin_3)
- net AUDIO_RIGHT: now also JTOP2.2 (Pin_2)
- net CLK: now also JTOP1.10 (Pin_10)
- net G0: now also JTOP1.1 (Pin_1)
- net G1: now also JTOP1.2 (Pin_2)
- net G2: now also JTOP1.3 (Pin_3)
- net G3: now also JTOP1.4 (Pin_4)
- net G4: now also JTOP1.5 (Pin_5)
- net G5: now also JTOP1.6 (Pin_6)
- net G6: now also JTOP1.7 (Pin_7)
- net G7: now also JTOP1.8 (Pin_8)
- net GND: now also JPICKIT1.3 (Pin_3), JTOP1.9 (Pin_9), JTOP2.4 (Pin_4)
- net HSOUT: now also JTOP2.9 (Pin_9)
- net ICSPCLK: now also JPICKIT1.5 (Pin_5)
- net ICSPDAT: now also JPICKIT1.4 (Pin_4)
- net SCL: now also JTOP2.7 (Pin_7)
- net SDA: now also JTOP2.6 (Pin_6)
- net VPP: now also JPICKIT1.1 (Pin_1)
- net VSOUT: now also JTOP2.8 (Pin_8)
- net BUTTON: now reaches U8.8 (PB4C)
- net BUTTON: now also JTOP2.10 (Pin_10)
- no-connect marks 13 -> 12

Commit message: PCB layout
Parts:
- removed JPICKIT1: Conn_01x05, Connector_PinHeader_2.54mm:PinHeader_1x05_P2.54mm_Vertical, symbol Connector_Generic:Conn_01x05
- added JPICKIT1: Conn_01x03, Connector_PinHeader_2.54mm:PinHeader_1x03_P2.54mm_Vertical, symbol Connector_Generic:Conn_01x03
- added JPICKIT2: Conn_01x02, Connector_PinHeader_2.54mm:PinHeader_1x02_P2.54mm_Vertical, symbol Connector_Generic:Conn_01x02
- R10, R11, R12, R13, R14, R15, R16, R17, R18, R19, R20, R21, R22, R23, R24, R25, R6, R7, R8, R9: footprint Resistor_SMD:R_0805_2012Metric -> Resistor_SMD:R_0603_1608Metric
Connections:
- net +3.3V: now also JPICKIT2.1 (Pin_1)
- net BLUE: now also R10.2, R11.2, R23.2, R7.2, R8.2, R9.2; no longer R17.2, R18.2, R19.2, R20.2, R21.2, R25.2
- net GND: now also JPICKIT1.2 (Pin_2)
- net ICSPCLK: now also JPICKIT1.1 (Pin_1)
- net ICSPDAT: now also JPICKIT1.3 (Pin_3)
- net RED: now also R17.2, R18.2, R19.2, R20.2, R21.2, R25.2; no longer R10.2, R11.2, R23.2, R7.2, R8.2, R9.2
- net VPP: now also JPICKIT2.2 (Pin_2)

Commit message: Squeeze all components onto the PCB
Parts:
- added C20: 100nF, Capacitor_SMD:C_0603_1608Metric, symbol Device:C_Small
Connections:
- net +3.3V: now also C20.1
- net BUTTON: now also U8.28 (PT12C); no longer U8.8 (PB4C)
- net CLK: now also U8.14 (PB11B); no longer U8.21 (PR5C)
- net G0: now also U8.4 (PL9A); no longer U8.13 (PB11A)
- net G1: now also U8.5 (PL9B); no longer U8.14 (PB11B)
- net G2: now also U8.8 (PB4C); no longer U8.16 (PB20C)
- net G3: now also U8.9 (PB6C); no longer U8.17 (PB20D)
- net G4: now also U8.10 (PB6D); no longer U8.20 (PR5D)
- net G5: now also U8.11 (PB9A); no longer U8.23 (DONE)
- net G6: now also U8.12 (PB9B); no longer U8.25 (PROGRAM)
- net G7: now also U8.13 (PB11A); no longer U8.26 (JTAGENB)
- net GND: now also C20.2
- net RCLK: now also U8.17 (PB20D); no longer U8.9 (PB6C)
- net SCL: now also U8.25 (PROGRAM); no longer U8.5 (PL9B)
- net SDA: now also U8.23 (DONE); no longer U8.4 (PL9A)
- net SER1: now also U8.16 (PB20C); no longer U8.12 (PB9B)
- net SER2: now also U8.21 (PR5C); no longer U8.11 (PB9A)
- net SRCLK: now also U8.20 (PR5D); no longer U8.10 (PB6D)
- net VSOUT: now also U8.26 (JTAGENB); no longer U8.28 (PT12C)
Changed lines of the file:
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@@
   (junction (at 128.27 176.53) (diameter 0) (color 0 0 0 0)
+  )
+  (junction (at 161.925 151.13) (diameter 0) (color 0 0 0 0)
   )
   (junction (at 128.27 153.67) (diameter 0) (color 0 0 0 0)
@@
     (stroke (width 0) (type default) (color 0 0 0 0))
   )
-  (wire (pts (xy 149.86 151.13) (xy 154.94 151.13))
+  (wire (pts (xy 149.86 151.13) (xy 161.925 151.13))
     (stroke (width 0) (type default) (color 0 0 0 0))
   )
@@
     (stroke (width 0) (type default) (color 0 0 0 0))
   )
+  (wire (pts (xy 161.925 151.13) (xy 161.925 151.765))
+    (stroke (width 0) (type default) (color 0 0 0 0))
+  )
   (wire (pts (xy 195.58 110.49) (xy 199.39 110.49))
     (stroke (width 0) (type default) (color 0 0 0 0))
@@
     (stroke (width 0) (type default) (color 0 0 0 0))
   )
-  (wire (pts (xy 118.11 124.46) (xy 118.11 109.22))
+  (wire (pts (xy 118.11 119.38) (xy 118.11 109.22))
     (stroke (width 0) (type default) (color 0 0 0 0))
   )
@@
     (stroke (width 0) (type default) (color 0 0 0 0))
   )
+  (wire (pts (xy 161.925 151.13) (xy 168.91 151.13))
+    (stroke (width 0) (type default) (color 0 0 0 0))
+  )
   (wire (pts (xy 147.32 95.25) (xy 156.21 95.25))
     (stroke (width 0) (type default) (color 0 0 0 0))
@@
     (stroke (width 0) (type default) (color 0 0 0 0))
   )
+  (wire (pts (xy 161.925 161.29) (xy 149.86 161.29))
+    (stroke (width 0) (type default) (color 0 0 0 0))
+  )
   (wire (pts (xy 78.74 86.36) (xy 90.17 86.36))
     (stroke (width 0) (type default) (color 0 0 0 0))
@@
     (stroke (width 0) (type default) (color 0 0 0 0))
   )
+  (wire (pts (xy 161.925 156.845) (xy 161.925 161.29))
+    (stroke (width 0) (type default) (color 0 0 0 0))
+  )
   (wire (pts (xy 185.42 46.99) (xy 185.42 44.45))
     (stroke (width 0) (type default) (color 0 0 0 0))
@@
     (stroke (width 0) (type default) (color 0 0 0 0))
   )
-  (label "G4" (at 110.49 59.69 270)
+  (label "G4" (at 137.16 96.52 180)
     (effects (font (size 1.27 1.27)) (justify right bottom))
   )
@@
     (effects (font (size 1.27 1.27)) (justify left bottom))
   )
-  (label "SER2" (at 137.16 93.98 180)
+  (label "SER2" (at 107.95 59.69 270)
     (effects (font (size 1.27 1.27)) (justify right bottom))
   )
@@
     (effects (font (size 1.27 1.27)) (justify right bottom))
   )
-  (label "VSOUT" (at 78.74 88.9 0)
-    (effects (font (size 1.27 1.27)) (justify left bottom))
-  )
-  (label "SRCLK" (at 137.16 96.52 180)
+  (label "VSOUT" (at 78.74 83.82 0)
+    (effects (font (size 1.27 1.27)) (justify left bottom))
+  )
+  (label "SRCLK" (at 110.49 59.69 270)
     (effects (font (size 1.27 1.27)) (justify right bottom))
   )
@@
     (effects (font (size 1.27 1.27)) (justify right bottom))
   )
-  (label "G3" (at 118.11 59.69 270)
+  (label "G3" (at 137.16 99.06 180)
     (effects (font (size 1.27 1.27)) (justify right bottom))
   )
@@
     (effects (font (size 1.27 1.27)) (justify left bottom))
   )
-  (label "G5" (at 102.87 59.69 270)
+  (label "G5" (at 137.16 93.98 180)
     (effects (font (size 1.27 1.27)) (justify right bottom))
   )
@@
     (effects (font (size 1.27 1.27)) (justify right bottom))
   )
-  (label "SCL" (at 110.49 119.38 90)
+  (label "SCL" (at 78.74 81.28 0)
     (effects (font (size 1.27 1.27)) (justify left bottom))
   )
@@
     (effects (font (size 1.27 1.27)) (justify right bottom))
   )
-  (label "G1" (at 137.16 86.36 180)
-    (effects (font (size 1.27 1.27)) (justify right bottom))
+  (label "G1" (at 110.49 119.38 90)
+    (effects (font (size 1.27 1.27)) (justify left bottom))
   )
   (label "TMS" (at 49.53 17.78 270)
@@
     (effects (font (size 1.27 1.27)) (justify right bottom))
   )
-  (label "SER1" (at 137.16 91.44 180)
+  (label "SER1" (at 137.16 81.28 180)
     (effects (font (size 1.27 1.27)) (justify right bottom))
   )
@@
     (effects (font (size 1.27 1.27)) (justify left bottom))
   )
-  (label "G7" (at 78.74 83.82 0)
-    (effects (font (size 1.27 1.27)) (justify left bottom))
+  (label "G7" (at 137.16 88.9 180)
+    (effects (font (size 1.27 1.27)) (justify right bottom))
   )
   (label "GREEN" (at 226.06 80.01 0)
@@
     (effects (font (size 1.27 1.27)) (justify right bottom))
   )
-  (label "SDA" (at 107.95 119.38 90)
-    (effects (font (size 1.27 1.27)) (justify left bottom))
+  (label "SDA" (at 102.87 59.69 270)
+    (effects (font (size 1.27 1.27)) (justify right bottom))
   )
   (label "SER2" (at 148.59 87.63 0)
@@
     (effects (font (size 1.27 1.27)) (justify left bottom))
   )
-  (label "G2" (at 137.16 81.28 180)
-    (effects (font (size 1.27 1.27)) (justify right bottom))
-  )
-  (label "G6" (at 78.74 81.28 0)
-    (effects (font (size 1.27 1.27)) (justify left bottom))
+  (label "G2" (at 118.11 119.38 90)
+    (effects (font (size 1.27 1.27)) (justify left bottom))
+  )
+  (label "G6" (at 137.16 91.44 180)
+    (effects (font (size 1.27 1.27)) (justify right bottom))
   )
   (label "BUTTON" (at 123.19 34.29 90)
@@
     (effects (font (size 1.27 1.27)) (justify left bottom))
   )
-  (label "BUTTON" (at 118.11 124.46 90)
-    (effects (font (size 1.27 1.27)) (justify left bottom))
-  )
-  (label "RCLK" (at 137.16 99.06 180)
-    (effects (font (size 1.27 1.27)) (justify right bottom))
-  )
-  (label "CLK" (at 107.95 59.69 270)
+  (label "BUTTON" (at 78.74 88.9 0)
+    (effects (font (size 1.27 1.27)) (justify left bottom))
+  )
+  (label "RCLK" (at 118.11 59.69 270)
+    (effects (font (size 1.27 1.27)) (justify right bottom))
+  )
+  (label "CLK" (at 137.16 86.36 180)
     (effects (font (size 1.27 1.27)) (justify right bottom))
   )
@@
     (effects (font (size 1.27 1.27)) (justify right bottom))
   )
-  (label "G0" (at 137.16 88.9 180)
-    (effects (font (size 1.27 1.27)) (justify right bottom))
+  (label "G0" (at 107.95 119.38 90)
+    (effects (font (size 1.27 1.27)) (justify left bottom))
   )
   (label "VSOUT" (at 118.11 34.29 90)
@@
     (pin "2")
   )
+  (symbol (lib_id "Device:C_Small") (at 161.925 154.305 0) (unit 1)
+    (in_bom yes) (on_board yes) (fields_autoplaced)
+    (property "Reference" "C20" (id 0) (at 165.1 153.0412 0)
+      (effects (font (size 1.27 1.27)) (justify left))
+    )
+    (property "Value" "100nF" (id 1) (at 165.1 155.5812 0)
+      (effects (font (size 1.27 1.27)) (justify left))
+    )
+    (property "Footprint" "Capacitor_SMD:C_0603_1608Metric" (id 2) (at 161.925 154.305 0)
+      (effects (font (size 1.27 1.27)) hide)
+    )
+    (property "Datasheet" "~" (id 3) (at 161.925 154.305 0)
+      (effects (font (size 1.27 1.27)) hide)
+    )
+    (pin "1")
+    (pin "2")
+  )
   (symbol (lib_id "Device:C_Small") (at 149.86 177.8 0) (unit 1)
     (in_bom yes) (on_board yes) (fields_autoplaced)
@@
     (pin "2")
   )
-  (symbol (lib_id "power:+3.3V") (at 154.94 151.13 270) (unit 1)
-    (in_bom yes) (on_board yes) (fields_autoplaced)
-    (property "Reference" "#PWR082" (id 0) (at 151.13 151.13 0)
-      (effects (font (size 1.27 1.27)) hide)
-    )
-    (property "Value" "+3.3V" (id 1) (at 158.75 151.1299 90)
+  (symbol (lib_id "power:+3.3V") (at 168.91 151.13 270) (unit 1)
+    (in_bom yes) (on_board yes) (fields_autoplaced)
+    (property "Reference" "#PWR082" (id 0) (at 165.1 151.13 0)
+      (effects (font (size 1.27 1.27)) hide)
+    )
+    (property "Value" "+3.3V" (id 1) (at 172.72 151.1299 90)
       (effects (font (size 1.27 1.27)) (justify left))
     )
-    (property "Footprint" "" (id 2) (at 154.94 151.13 0)
-      (effects (font (size 1.27 1.27)) hide)
-    )
-    (property "Datasheet" "" (id 3) (at 154.94 151.13 0)
-      (effects (font (size 1.27 1.27)) hide)
-    )
+    (property "Footprint" "" (id 2) (at 168.91 151.13 0)
+      (effects (font (size 1.27 1.27)) hide)
+    )
+    (property "Datasheet" "" (id 3) (at 168.91 151.13 0)
+      (effects (font (size 1.27 1.27)) hide)
+    )
