File: signalgenerator/board/board.kicad_pcb (KiCad board)
At the start: 2 copper layers, 37.5 x 23 mm, 20 parts, among them J1 Barrel_Jack_Switch, SW1 SW_DIP_x04, U1 MIC5504-3.3YM5, U2 XO2-DIP20, U3 74LVC04, X1 ASE-80MHz

Commit message: Implement NES signal PAL/NTSC
Parts:
- removed C5: 100nF, Capacitor_SMD:C_0603_1608Metric_Pad1.08x0.95mm_HandSolder
- removed X1: ASE-80MHz, Oscillator:Oscillator_SMD_Abracon_ASE-4Pin_3.2x2.5mm
- added X2: XO53, Oscillator:Oscillator_SMD_EuroQuartz_XO53-4Pin_5.0x3.2mm, F.Cu at (145.7, 131.4)
- U1: value MIC5504-3.3YM5 -> AMS1117-3.3; footprint Package_TO_SOT_SMD:SOT-23-5 -> Package_TO_SOT_SMD:SOT-223-3_TabPin2
- moved U3 25.6 mm to (138.0, 132.2), turned to 0 degrees
- moved U1 16.5 mm to (138.6, 124.8), turned to 0 degrees
Connections:
- C1 pad 1: Net-(U1-EN) -> Net-(U1-VI)
- J1 pad 1: Net-(U1-EN) -> Net-(U1-VI)
- U1 pad 1: Net-(U1-EN) -> GND
- U1 pad 2: GND -> +3.3V
- U1 pad 3: Net-(U1-EN) -> Net-(U1-VI)
- U3 pad 14: unconnected-(U3-VCC-Pad14) -> +3.3V
Routing:
- net Net-(U1-VI): track 0.00 -> 15.6 mm
- net Net-(U1-EN): track 15.6 -> 0.00 mm
