File: testrig/board/board.kicad_sch (KiCad schematic)
At the start: 17 parts, among them J1 Conn_01x20, J2 Conn_01x20, SW1 SW_DIP_x01, SW2 SW_DIP_x01, U1 AMS1117-3.3, U2 XO2-DIP20, U3 74HC574, U4 74HC574, U5 74HC574, U6 74HC574

Commit message: Rewire mode switch in rest rig
Parts:
- removed R1: 10k, symbol Device:R_Small
- removed SW2: SW_DIP_x01, symbol Switch:SW_DIP_x01
- added JP1: Jumper_2_Open, symbol Jumper:Jumper_2_Open
Connections:
- net +3.3V: now also JP1.2 (B)
- net at U2.17 (PIN26): now also JP1.1 (A)
